Commit message: feat: Stability Fix
Modified my urdf file to eliminate robot instability. Will turn this project in and receive feedback from reviewer.

File: src/my_robot/urdf/my_robot.xacro (robot description, xacro)
@@ -9,5 +9,5 @@
   </joint>
   <joint type="continuous" name="left_wheel_hinge">
-    <origin xyz="0 0.15 0" rpy="0 0 0"/>
+    <origin xyz=".0 0.15 .0" rpy="0 0 0"/>
     <child link="left_wheel"/>
     <parent link="chassis"/>
@@ -17,5 +17,5 @@
   </joint>
   <joint type="continuous" name="right_wheel_hinge">
-    <origin xyz="0 -0.15 0" rpy="0 0 0"/>
+    <origin xyz=".0 -0.15 .0" rpy="0 0 0"/>
     <child link="right_wheel"/>
     <parent link="chassis"/>
@@ -25,5 +25,5 @@
   </joint>
   <joint type="fixed" name="camera_joint">
-    <origin xyz=".2 0 .1" rpy="0 0 0"/>
+    <origin xyz=".25 0 0" rpy="0 0 0"/>
     <child link="camera"/>
     <parent link="chassis"/>
@@ -31,5 +31,5 @@
   </joint>
   <joint type="fixed" name="hokuyo_joint">
-    <origin xyz=".15 0 .2" rpy="0 0 0"/>
+    <origin xyz=".2 0 .1" rpy="0 0 0"/>
     <child link="hokuyo"/>
     <parent link="chassis"/>
@@ -37,7 +37,7 @@
   </joint>
   <link name='chassis'>
-    <pose>0 0 0.2 0 0 0</pose>
+    <pose>0 0 0.1 0 0 0</pose>
     <inertial>
-      <mass value="15.0"/>
+      <mass value="35.0"/>
       <origin xyz="0 0 0" rpy=" 0 0 0"/>
       <inertia
@@ -50,5 +50,5 @@
       <origin xyz="0 0 0" rpy=" 0 0 0"/>
       <geometry>
-        <box size=".4 .2 .3"/>
+        <box size=".5 .2 .1"/>
       </geometry>
     </collision>
@@ -56,29 +56,29 @@
       <origin xyz="0 0 0" rpy=" 0 0 0"/>
       <geometry>
-        <box size=".4 .2 .3"/>
+        <box size=".5 .2 .1"/>
       </geometry>
     </visual>
     <collision name='back_caster_collision'>
-      <origin xyz="-0.2 0 -0.1" rpy=" 0 0 0"/>
+      <origin xyz="-0.15 0 -0.05" rpy=" 0 0 0"/>
       <geometry>
-        <sphere radius="0.085"/>
+        <sphere radius="0.0499"/>
       </geometry>
     </collision>
     <visual name='back_caster_visual'>
-      <origin xyz="-0.2 0 -0.1" rpy=" 0 0 0"/>
+      <origin xyz="-0.15 0 -0.05" rpy=" 0 0 0"/>
       <geometry>
-        <sphere radius="0.085"/>
+        <sphere radius="0.05"/>
       </geometry>
     </visual>
     <collision name='front_caster_collision'>
-      <origin xyz="0.15 0 -0.1" rpy=" 0 0 0"/>
+      <origin xyz="0.15 0 -0.05" rpy=" 0 0 0"/>
       <geometry>
-        <sphere radius="0.085"/>
+        <sphere radius="0.0499"/>
       </geometry>
     </collision>
     <visual name='front_caster_visual'>
-      <origin xyz="0.15 0 -0.1" rpy=" 0 0 0"/>
+      <origin xyz="0.15 0 -0.05" rpy=" 0 0 0"/>
       <geometry>
-        <sphere radius="0.085"/>
+        <sphere radius="0.05"/>
       </geometry>
     </visual>
@@ -96,5 +96,5 @@
     <collision name='collision'>
       <geometry>
-        <cylinder radius=".2" length=".05"/>
+        <cylinder radius=".1" length=".1"/>
       </geometry>
       <origin xyz="0 0 0" rpy="0 1.5707 1.5707"/>
@@ -102,5 +102,5 @@
     <visual name='visual'>
       <geometry>
-        <cylinder radius=".2" length=".05"/>
+        <cylinder radius=".1" length=".1"/>
       </geometry>
       <origin xyz="0 0 0" rpy="0 1.5707 1.5707"/>
@@ -119,5 +119,5 @@
     <collision name='collision'>
       <geometry>
-        <cylinder radius=".2" length=".05"/>
+        <cylinder radius=".1" length=".1"/>
       </geometry>
       <origin xyz="0 0 0" rpy="0 1.5707 1.5707"/>
@@ -125,5 +125,5 @@
     <visual name='visual'>
       <geometry>
-        <cylinder radius=".2" length=".05"/>
+        <cylinder radius=".1" length=".1"/>
       </geometry>
       <origin xyz="0 0 0" rpy="0 1.5707 1.5707"/>
